File: badge_template/badge_template.kicad_pcb (KiCad board)
At the start: 2 copper layers, 59.9 x 81 mm, 15 parts

Commit message: update: pcb update
Parts:
- removed ? (x2): , 
- added G***: LOGO, LOGO, F.Cu at (123.1, 146.2)
- added G***: LOGO, LOGO, F.Cu at (134.5, 115.8)
- D5, D6, R5, R6: moved to F.Cu
- moved D1 13.0 mm to (141.0, 139.0), turned to 90 degrees
- moved D4 13.0 mm to (128.0, 139.0)
- moved R4 13.0 mm to (128.0, 134.0)
- moved R1 13.0 mm to (141.0, 134.0)
- moved D2 4.51 mm to (137.0, 139.0)
- moved D3 4.51 mm to (132.5, 139.0)
- moved R3 4.50 mm to (132.5, 134.0)
- moved R2 4.50 mm to (137.0, 133.9)
- moved D6 4.00 mm to (120.0, 92.5)
- moved R6 4.00 mm to (120.0, 89.2), turned to 0 degrees
- moved D5 3.51 mm to (149.5, 92.5)
- moved R5 3.51 mm to (149.5, 89.0), turned to 180 degrees
Routing:
- net Net-(D1-K): track 0.00 -> 101.1 mm, vias 0 -> 6
- net Net-(A1-D5): track 0.00 -> 43.7 mm, vias 0 -> 1
- net Net-(A1-D4): track 0.00 -> 37.1 mm, vias 0 -> 1
- net Net-(A1-D3): track 0.00 -> 30.4 mm, vias 0 -> 1
- net Net-(A1-D2): track 0.00 -> 26.2 mm, vias 0 -> 1
- net Net-(A1-D9): track 0.00 -> 22.3 mm, vias 0 -> 1
- net Net-(A1-D8): track 0.00 -> 8.58 mm, vias 0 -> 1
- net Net-(D3-A): track 0.00 -> 3.95 mm, vias 0 -> 2
- net Net-(D4-A): track 0.00 -> 3.93 mm, vias 0 -> 2
- net Net-(D2-A): track 0.00 -> 3.89 mm, vias 0 -> 2
- net Net-(D1-A): track 0.00 -> 3.89 mm, vias 0 -> 2
- net Net-(D5-A): track 0.00 -> 2.85 mm, vias 0 -> 2
- net Net-(D6-A): track 0.00 -> 2.67 mm, vias 0 -> 2
Other:
- board size 59.9 x 81 mm -> 59.9 x 78.7 mm
- board text added: "덕영고등학교"
- board text added: "덕영고등학교 소프트웨어부"

Commit message: update: pcb update
Parts:
- removed A1: Arduino_Nano_v2.x, Module:Arduino_Nano
- added A2: Arduino_Nano_v3.x, Module:Arduino_Nano, F.Cu at (142.2, 118.1)
- R1, R2, R3, R4, R5, R6: value 47 -> 130
