File: badge_template/badge_template.kicad_sch (KiCad schematic)
At the start: 13 parts

Commit message: update: pcb update
Parts:
- R1, R2, R3, R4, R5, R6: value 47 -> 130
Changed lines of the file:
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@@
 			)
 		)
-		(property "Value" "47"
+		(property "Value" "130"
 			(at 89.154 99.06 0)
 			(effects
@@
 			)
 		)
-		(property "Value" "47"
+		(property "Value" "130"
 			(at 89.154 92.71 0)
 			(effects
@@
 			)
 		)
-		(property "Value" "47"
+		(property "Value" "130"
 			(at 89.154 80.01 0)
 			(effects
@@
 			)
 		)
-		(property "Value" "47"
+		(property "Value" "130"
 			(at 95.504 104.14 0)
 			(effects
@@
 			)
 		)
-		(property "Value" "47"
+		(property "Value" "130"
 			(at 95.504 109.22 0)
 			(effects
@@
 			)
 		)
-		(property "Value" "47"
+		(property "Value" "130"
 			(at 89.154 86.36 0)
 			(effects

Commit message: update: pcb update
Parts:
- removed A1: Arduino_Nano_v2.x, Module:Arduino_Nano, symbol MCU_Module:Arduino_Nano_v2.x
- added A2: Arduino_Nano_v3.x, Module:Arduino_Nano, symbol MCU_Module:Arduino_Nano_v3.x
Connections:
- net at R4.2: now also A2.8 (D5)
- net at R3.2: now also A2.7 (D4)
- net at D1.1 (K), D2.1 (K), D3.1 (K)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: now also A2.4 (GND)
- net at R1.2: now also A2.5 (D2)
- net at R5.2: now also A2.11 (D8)
- net at R6.2: now also A2.12 (D9)
- net at R2.2: now also A2.6 (D3)
Changed lines of the file:
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@@
+	)
+	(junction
+		(at 124.46 119.38)
+		(diameter 0)
+		(color 0 0 0 0)
 	)
 	(junction
 		(at 74.93 96.52)
-		(diameter 0)
-		(color 0 0 0 0)
-	)
-	(junction
-		(at 124.46 119.38)
 		(diameter 0)
 		(color 0 0 0 0)
@@
 	)
 	(symbol
+		(lib_id "MCU_Module:Arduino_Nano_v3.x")
+		(at 124.46 93.98 0)
+		(unit 1)
+		(exclude_from_sim no)
+		(in_bom yes)
+		(on_board yes)
+		(dnp no)
+		(fields_autoplaced yes)
+		(property "Reference" "A2"
+			(at 129.1941 119.38 0)
+			(effects
+				(font
+					(size 1.27 1.27)
+				)
+				(justify left)
+			)
+		)
+		(property "Value" "Arduino_Nano_v3.x"
+			(at 129.1941 121.92 0)
+			(effects
+				(font
+					(size 1.27 1.27)
+				)
+				(justify left)
+			)
+		)
+		(property "Footprint" "Module:Arduino_Nano"
+			(at 124.46 93.98 0)
+			(effects
+				(font
+					(size 1.27 1.27)
+					(italic yes)
+				)
+				(hide yes)
+			)
+		)
+		(property "Datasheet" "http://www.mouser.com/pdfdocs/Gravitech_Arduino_Nano3_0.pdf"
+			(at 124.46 93.98 0)
+			(effects
+				(font
+					(size 1.27 1.27)
+				)
+				(hide yes)
+			)
+		)
+		(property "Description" "Arduino Nano v3.x"
+			(at 124.46 93.98 0)
+			(effects
+				(font
+					(size 1.27 1.27)
+				)
+				(hide yes)
+			)
+		)
+		(pin "13"
+		)
+		(pin "27"
+		)
+		(pin "30"
+		)
+		(pin "2"
+		)
+		(pin "10"
+		)
+		(pin "29"
+		)
+		(pin "16"
+		)
+		(pin "9"
+		)
+		(pin "7"
+		)
+		(pin "3"
+		)
+		(pin "23"
+		)
+		(pin "14"
+		)
+		(pin "6"
+		)
+		(pin "18"
+		)
+		(pin "24"
+		)
+		(pin "26"
+		)
+		(pin "17"
+		)
+		(pin "11"
+		)
+		(pin "28"
+		)
+		(pin "25"
+		)
+		(pin "1"
+		)
+		(pin "8"
+		)
+		(pin "22"
+		)
+		(pin "19"
+		)
+		(pin "20"
+		)
+		(pin "4"
+		)
+		(pin "12"
+		)
+		(pin "5"
+		)
+		(pin "21"
+		)
+		(pin "15"
+		)
+		(instances
+			(project ""
+				(path "/7966b607-d2b7-4f48-a4fc-a876c3848eb5"
+					(reference "A2")
+					(unit 1)
+				)
+			)
+		)
+	)
+	(symbol
 		(lib_id "Device:R")
 		(at 96.52 113.03 90)
@@
 					(unit 1)
 				)
-			)
-		)
-	)
-	(symbol
-		(lib_id "MCU_Module:Arduino_Nano_v2.x")
-		(at 124.46 93.98 0)
-		(unit 1)
-		(exclude_from_sim no)
-		(in_bom yes)
-		(on_board yes)
-		(dnp no)
-		(fields_autoplaced yes)
-		(property "Reference" "A1"
-			(at 129.1941 119.38 0)
-			(effects
-				(font
-					(size 1.27 1.27)
-				)
-				(justify left)
-			)
-		)
-		(property "Value" "Arduino_Nano_v2.x"
-			(at 129.1941 121.92 0)
-			(effects
-				(font
-					(size 1.27 1.27)
-				)
-				(justify left)
-			)
-		)
-		(property "Footprint" "Module:Arduino_Nano"
-			(at 124.46 93.98 0)
-			(effects
-				(font
-					(size 1.27 1.27)
-					(italic yes)
-				)
-				(hide yes)
-			)
-		)
-		(property "Datasheet" "https://www.arduino.cc/en/uploads/Main/ArduinoNanoManual23.pdf"
-			(at 124.46 93.98 0)
-			(effects
-				(font
-					(size 1.27 1.27)
-				)
-				(hide yes)
-			)
-		)
-		(property "Description" "Arduino Nano v2.x"
-			(at 124.46 93.98 0)
-			(effects
-				(font
-					(size 1.27 1.27)
-				)
-				(hide yes)
-			)
-		)
-		(pin "12"
-		)
-		(pin "14"
-		)
-		(pin "19"
-		)
-		(pin "23"
-		)
-		(pin "1"
-		)
-		(pin "29"
-		)
-		(pin "3"
-		)
-		(pin "7"
-		)
-		(pin "8"
-		)
-		(pin "20"
-		)
-		(pin "16"
-		)
-		(pin "9"
-		)
-		(pin "30"
-		)
-		(pin "10"
-		)
-		(pin "26"
-		)
-		(pin "24"
-		)
-		(pin "11"
-		)
-		(pin "18"
-		)
-		(pin "28"
-		)
-		(pin "6"
-		)
-		(pin "15"
-		)
-		(pin "17"
-		)
-		(pin "2"
-		)
-		(pin "21"
-		)
-		(pin "22"
-		)
-		(pin "25"
-		)
-		(pin "27"
-		)
-		(pin "4"
-		)
-		(pin "5"
-		)
-		(pin "13"
-		)
-		(instances
-			(project ""
-				(path "/7966b607-d2b7-4f48-a4fc-a876c3848eb5"
-					(reference "A1")
-					(unit 1)
-				)
